File: schematics/v1_ordered/onion_dip_v1.sch (EAGLE design)
At the start: 38 parts, among them IC2 DS2432P

Commit message: added sch pdf
Other:
- note added: "Connectors"
- note added: "LEDs"
- note added: "Logos"
- note added: "Power"
- moved on the sheet: ASDASD, GND, IC2, IC2P, IC2_1W, JP3, LED1, LED2, LED5, R1, R2, R3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
